Commit message: 初始提交2

File: src/robotic_arm/model/robotic_arm.urdf (robot description, URDF)
Before this commit: robot robotic_arm, 7 links, 6 joints
Links:
- link base_link: geometry collision mesh filename=base_link.STL; visual mesh filename=base_link.STL
- link link1: geometry collision mesh filename=link1.STL; visual mesh filename=link1.STL
- link link2: geometry collision mesh filename=link2.STL; visual mesh filename=link2.STL
- link link3: geometry collision mesh filename=link3.STL; visual mesh filename=link3.STL
- link link4: geometry collision mesh filename=link4.STL; visual mesh filename=link4.STL
- link link5: geometry collision mesh filename=link5.STL; visual mesh filename=link5.STL
- link link6: geometry collision mesh filename=link6.STL; visual mesh filename=link6.STL

File: src/robotic_config/config/robotic_arm.ros2_control.xacro (robot description, xacro)
@@ -1,66 +1,15 @@
 <?xml version="1.0"?>
 <robot xmlns:xacro="http://www.ros.org/wiki/xacro">
-    <xacro:macro name="robotic_arm_ros2_control" params="name initial_positions_file">
-        <xacro:property name="initial_positions" value="${load_yaml(initial_positions_file)['initial_positions']}"/>
-        <ros2_control name="${name}" type="system">
-            <hardware>
-                <!-- By default, set up controllers for simulation. This won't work on real hardware -->
-                <plugin>mock_components/GenericSystem</plugin>
-            </hardware>
-            <joint name="joint1">
-                <command_interface name="position"/>
-                <command_interface name="velocity"/>
-                <command_interface name="effort"/>
-                <state_interface name="position">
-                  <param name="initial_value">${initial_positions['joint1']}</param>
-                </state_interface>
-                <state_interface name="velocity"/>
-            </joint>
-            <joint name="joint2">
-                <command_interface name="position"/>
-                <command_interface name="velocity"/>
-                <command_interface name="effort"/>
-                <state_interface name="position">
-                  <param name="initial_value">${initial_positions['joint2']}</param>
-                </state_interface>
-                <state_interface name="velocity"/>
-            </joint>
-            <joint name="joint3">
-                <command_interface name="position"/>
-                <command_interface name="velocity"/>
-                <command_interface name="effort"/>
-                <state_interface name="position">
-                  <param name="initial_value">${initial_positions['joint3']}</param>
-                </state_interface>
-                <state_interface name="velocity"/>
-            </joint>
-            <joint name="joint4">
-                <command_interface name="position"/>
-                <command_interface name="velocity"/>
-                <command_interface name="effort"/>
-                <state_interface name="position">
-                  <param name="initial_value">${initial_positions['joint4']}</param>
-                </state_interface>
-                <state_interface name="velocity"/>
-            </joint>
-            <joint name="joint5">
-                <command_interface name="position"/>
-                <command_interface name="velocity"/>
-                <command_interface name="effort"/>
-                <state_interface name="position">
-                  <param name="initial_value">${initial_positions['joint5']}</param>
-                </state_interface>
-                <state_interface name="velocity"/>
-            </joint>
-            <joint name="joint6">
-                <command_interface name="position"/>
-                <command_interface name="velocity"/>
-                <command_interface name="effort"/>
-                <state_interface name="position">
-                  <param name="initial_value">${initial_positions['joint6']}</param>
-                </state_interface>
-                <state_interface name="velocity"/>
-            </joint>
-        </ros2_control>
+    <xacro:include filename="robotic_arm_real.urdf.xacro" />
+    <xacro:include filename="robotic_arm_mujoco.urdf.xacro" />
+    <xacro:macro name="robotic_arm_ros2_control" params="backend name initial_positions_file">
+        <xacro:if value="${backend == 'real'}">
+            <xacro:robotic_arm_real_ros2_control name="${name}" />
+        </xacro:if>
+        <xacro:if value="${backend == 'mujoco'}">
+            <xacro:robotic_arm_mujoco_ros2_control
+                name="${name}"
+                initial_positions_file="${initial_positions_file}" />
+        </xacro:if>
     </xacro:macro>
 </robot>

File: src/robotic_config/config/robotic_arm.urdf.xacro (robot description, xacro)
@@ -1,9 +1,17 @@
 <?xml version="1.0"?>
 <robot xmlns:xacro="http://www.ros.org/wiki/xacro" name="robotic_arm">
-    <xacro:arg name="initial_positions_file" default="initial_positions.yaml" />
+    <xacro:arg name="backend" default="real" />
+    <xacro:arg name="initial_positions_file" default="$(find robotic_config)/config/initial_positions.yaml" />
+    <xacro:property name="backend" value="$(arg backend)" />
     <!-- Import robotic_arm urdf file -->
-    <xacro:include filename="$(find robotic_arm)/urdf/robotic_arm.urdf" />
+    <xacro:include filename="$(find robotic_arm)/robotic_arm.urdf" />
     <!-- Import control_xacro -->
     <xacro:include filename="robotic_arm.ros2_control.xacro" />
-    <xacro:robotic_arm_ros2_control name="FakeSystem" initial_positions_file="$(arg initial_positions_file)"/>
+    <xacro:if value="${backend == 'mujoco'}">
+        <xacro:robotic_arm_mujoco_config />
+    </xacro:if>
+    <xacro:robotic_arm_ros2_control
+        backend="${backend}"
+        name="arm_hw"
+        initial_positions_file="$(arg initial_positions_file)"/>
 </robot>

Commit message: 在Mujoco仿真环境中操作机械臂完成基本动作

File: src/robotic_arm/model/robotic_arm.urdf (robot description, URDF)
Before this commit: robot robotic_arm, 7 links, 6 joints
Links:
- link base_link: geometry collision mesh filename=package://robotic_arm/base_link.STL; visual mesh filename=package://robotic_arm/base_link.STL
- link link1: geometry collision mesh filename=package://robotic_arm/link1.STL; visual mesh filename=package://robotic_arm/link1.STL
- link link2: geometry collision mesh filename=package://robotic_arm/link2.STL; visual mesh filename=package://robotic_arm/link2.STL
- link link3: geometry collision mesh filename=package://robotic_arm/link3.STL; visual mesh filename=package://robotic_arm/link3.STL
- link link4: geometry collision mesh filename=package://robotic_arm/link4.STL; visual mesh filename=package://robotic_arm/link4.STL
- link link5: geometry collision mesh filename=package://robotic_arm/link5.STL; visual mesh filename=package://robotic_arm/link5.STL
- link link6: geometry collision mesh filename=package://robotic_arm/link6.STL; visual mesh filename=package://robotic_arm/link6.STL
Joints:
- joint joint6: origin xyz=0.073796 0.0036822 8.8922E-05 rpy=0 -1.5708 0 -> xyz=0.073796 0.0036822 8.8922E-05 rpy=0 -1.5708 3.14

File: src/robotic_config/config/robotic_arm_mujoco.urdf.xacro (robot description, xacro)
@@ -72,4 +72,8 @@
         <state_interface name="effort"/>
       </joint>
+      <gpio name="suction">
+        <command_interface name="vacuum" data_type="bool"/>
+        <state_interface name="vacuum" data_type="bool"/>
+      </gpio>
     </ros2_control>
   </xacro:macro>

File: src/robotic_config/config/robotic_arm_real.urdf.xacro (robot description, xacro)
@@ -54,4 +54,8 @@
         <state_interface name="effort"/>
       </joint>
+      <gpio name="suction">
+        <command_interface name="vacuum" data_type="bool"/>
+        <state_interface name="vacuum" data_type="bool"/>
+      </gpio>
     </ros2_control>
   </xacro:macro>

Commit message: 完成机械臂抓取动作流程的测试

File: src/robotic_arm/model/robotic_arm.urdf (robot description, URDF)
Before this commit: robot robotic_arm, 7 links, 6 joints
Joints:
- joint joint1: limit lower=-6.283185307 upper=6.283185307 effort=50 velocity=10 -> lower=-2.0 upper=2.0 effort=50 velocity=10
- joint joint3: limit lower=-3.141592654 upper=3.141592654 effort=50 velocity=10 -> lower=-2.8 upper=2.8 effort=50 velocity=10
- joint joint4: limit lower=-3.141592654 upper=3.141592654 effort=50 velocity=10 -> lower=-2.5 upper=2.5 effort=50 velocity=10
